File: cmm-4030d-breakout/cmm-4030d-breakout.kicad_pcb (KiCad board)
At the start: 2 copper layers, 25.4 x 25.4 mm, 13 parts, among them J1 Conn_01x07_Female

Commit message: pcb update
Other:
- rule pad_to_mask_clearance: 0 -> 0.0508
- rule via_min_drill: 0.5 -> 0.254
- rule via_min_size: 0.8 -> 0.508
- board text added: "0804-0601180901"
- board text added: "CE"
- board text added: "DOUT"
- board text added: "GND"
- board text added: "Left"
- board text added: "Right"
- board text added: "SCK"
- board text added: "SELECT"
- board text added: "VDD"
- board text added: "WS"
- board text added: "v0"
